File: hardware/project 1.kicad_sch (KiCad schematic)
At the start: 0 parts

Commit message: Add files via upload
Parts:
- added C1, C2: 10µF, Capacitor_SMD:C_0805_2012Metric, symbol Device:C
- added C3: C, Capacitor_SMD:C_0805_2012Metric, symbol Device:C
- added D1, D2, D3, D4: WS2812B, LED_SMD:LED_WS2812B_PLCC4_5.0x5.0mm_P3.2mm, symbol LED:WS2812B
- added H1, H2, H3, H4: MountingHole, Button_Switch_Keyboard:SW_Cherry_MX_2.25u_Plate, symbol Mechanical:MountingHole
- added J1: USB_C_Receptacle_USB2.0_14P, Connector_USB:USB_C_Receptacle_HRO_TYPE-C-31-M-12, symbol Connector:USB_C_Receptacle_USB2.0_14P
- added R1, R2: 5.1kΩ, Resistor_SMD:R_0805_2012Metric, symbol Device:R_US
- added R3: R_US, Resistor_SMD:R_0805_2012Metric, symbol Device:R_US
- added R4: 330Ω, Resistor_SMD:R_0805_2012Metric, symbol Device:R_US
- added SW1, SW2, SW3, SW4, SW5, SW6, SW7, SW8, SW9: SW_Push, Button_Switch_Keyboard:SW_Cherry_MX_1.00u_PCB, symbol Switch:SW_Push
- added SW10: RotaryEncoder_Switch, Rotary_Encoder:RotaryEncoder_Alps_EC12E-Switch_Vertical_H20mm, symbol Device:RotaryEncoder_Switch
- added U1: ESP32-S3-WROOM-1, RF_Module:ESP32-S3-WROOM-1, symbol RF_Module:ESP32-S3-WROOM-1
- added U2: AMS1117-3.3, Package_TO_SOT_SMD:SOT-223-3_TabPin2, symbol Regulator_Linear:AMS1117-3.3
- added U3: ER_OLEDM0.91_1x-I2C, Display:ER_OLEDM0.91_1x-I2C, symbol Display_Graphic:ER_OLEDM0.91_1x-I2C
Connections:
- new net: R4.1, U1.32 (IO39)
- new net: D1.4 (DIN), R4.2
- new net: U1.10 (IO17), U3.3 (SCL)
- new net: U1.11 (IO18), U3.4 (SDA)
- new net: C3.1, R3.1, U1.3 (EN)
- new net: J1.B5 (CC2), R2.1
- new net: J1.A5 (CC1), R1.1
- new net: J1.A7 (D-), U1.13 (USB_D-)
- new net: J1.B6 (D+), U1.14 (USB_D+)
- new net +3V3: C2.1, R3.2, U1.2 (3V3), U2.2 (VO), U3.2 (VCC)
- new net +5V: C1.1, D1.1 (VDD), D2.1 (VDD), D3.1 (VDD), D4.1 (VDD), J1.A4 (VBUS), J1.A9 (VBUS), J1.B4 (VBUS), J1.B9 (VBUS), U2.3 (VI)
- new net DOUT1: D1.2 (DOUT), D4.4 (DIN)
- new net DOUT2: D3.4 (DIN), D4.2 (DOUT)
- new net DOUT3: D2.4 (DIN), D3.2 (DOUT)
- new net GND: C1.2, C2.2, C3.2, D1.3 (VSS), D2.3 (VSS), D3.3 (VSS), D4.3 (VSS), J1.A1 (GND), J1.A12 (GND), J1.B1 (GND), J1.B12 (GND), R1.2, R2.2, SW1.2, SW10.C, SW10.S2, SW2.2, SW3.2, SW4.2, SW5.2, SW6.2, SW7.2, SW8.2, SW9.2, U1.1 (GND), U1.40 (GND), U1.41 (GND), U2.1 (GND), U3.1 (GND)
- new net IO1: SW1.1, U1.39 (IO1)
- new net IO10: SW10.S1, U1.18 (IO10)
- new net IO11: SW10.A, U1.19 (IO11)
- new net IO12: SW10.B, U1.20 (IO12)
- new net IO2: SW2.1, U1.38 (IO2)
- new net IO3: SW3.1, U1.15 (IO3)
- new net IO4: SW4.1, U1.4 (IO4)
- new net IO5: SW5.1, U1.5 (IO5)
- new net IO6: SW6.1, U1.6 (IO6)
- new net IO7: SW7.1, U1.7 (IO7)
- new net IO8: SW8.1, U1.12 (IO8)
- new net IO9: SW9.1, U1.17 (IO9)
- no-connect marks 0 -> 3
